File: TRRS/half-swept.kicad_pcb (KiCad board)
At the start: 2 copper layers, 109.4 x 86.9 mm, 27 parts, among them J2 AudioJack4dpb, SW1 SW_Push, SW10 SW_Push, SW11 SW_Push, SW12 SW_Push, SW13 SW_Push, SW14 SW_Push, SW15 SW_Push, SW16 SW_Push, SW17 SW_Push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

Commit message: new new new
Routing:
- net raw: track 55.6 -> 52.7 mm
