File: USB-C/K02-USB-C.kicad_sch (KiCad schematic)
At the start: 46 parts

Commit message: fixed
Parts:
- Bat+1, Bat+r1, BatGND1, BatGND4: value (none) -> MountingHole_Pad; footprint (none) -> kbd:1pin_conn
- J1, J2: value (none) -> AudioJack4dpb; footprint (none) -> kbd:MJ-4PP-9
- RSW1, RSW2: value (none) -> SW_Push; footprint (none) -> kbd:ResetSW
- SW10, SW10_r1, SW11, SW11_r1, SW12, SW12_r1, SW13_r1, SW14, SW14_r1, SW15, SW15_r1, SW16, SW16_r1, SW17, SW17_r1, SW18, SW18_r1, SW2, SW20, SW21, SW2_r1, SW3, SW3_r1, SW4, SW4_r1, SW5, SW5_r1, SW6, SW6_r1, SW7_r1, SW8, SW8_r1, SW9, SW9_r1: value (none) -> SW_Push; footprint (none) -> Kailh:SW_PG1350_rev_DPB
- SW_POWER1, SW_POWERR1: value (none) -> SW_SPDT; footprint (none) -> Kailh:SPDT_C128955
- U1, U2: value (none) -> ProMicro-kbd; footprint (none) -> kbd:ProMicro_v2
Other:
- note added: "TRRS but I'ts USB-C"
- company: broomlabs -> (none)
- title: Sweep V2 -> K02
